File: hardware/Qoobinoo_v2.0/Qoobinoo.kicad_pcb (KiCad board)
At the start: 2 copper layers, 54 x 84 mm, 32 parts, among them J1 USB_C_Receptacle_USB2.0, J2 Conn_01x02, J3 Conn_01x12, J4 Conn_01x12, SW1 SW_Push, SW2 SW_Push, U1 ATmega32U4-M, X1 16MHz

Commit message: Change USB
Parts:
- removed J1: USB_C_Receptacle_USB2.0, Moldex-21699:Molex-216990_GCT-USB45xx_HRO-TYPE-C-31-M-13x
- added P1: USB_C_Plug_USB2.0, Connector_USB:USB_C_Receptacle_CNCTech_C-ARA1-AK51X, F.Cu at (150.2, 55.3)
- C4, C8: footprint Resistor_SMD:R_1206_3216Metric -> Capacitor_SMD:C_1206_3216Metric
- J2: value Conn_01x02 -> Conn_01x02_Female; footprint Pin:Pins_USB -> Pin:Pins_1x02
- R4, R5: footprint Resistor_SMD:R_1206_3216Metric -> Resistor_SMD:R_0805_2012Metric
- moved J2 1.14 mm to (149.2, 62.7)
- turned D3 to 90 degrees
- turned D4 to 90 degrees
Connections:
- D3 pad 1: /PC6 -> Net-(D3-Pad1)
- D3 pad 2: Net-(D3-Pad2) -> /PC6
- D4 pad 1: /PC7 -> Net-(D4-Pad1)
- D4 pad 2: Net-(D4-Pad2) -> /PC7
- R2 pad 1: Net-(D3-Pad2) -> Net-(D3-Pad1)
- R3 pad 1: Net-(D4-Pad2) -> Net-(D4-Pad1)
Routing:
- net /D-: track 53.2 -> 48.5 mm, vias 2 -> 1
- net Net-(F1-Pad1): track 22.6 -> 27.1 mm
- net GND: track 72.0 -> 75.8 mm, vias 8 -> 44
- net /D+: track 53.3 -> 50.0 mm, vias 1 -> 2
- net Net-(D4-Pad2): track 2.80 -> 0.00 mm
- net Net-(D4-Pad1): track 0.00 -> 2.80 mm
- net Net-(D3-Pad2): track 2.75 -> 0.00 mm
- net Net-(D3-Pad1): track 0.00 -> 2.75 mm
- net /PD+: track 7.89 -> 8.44 mm
- net /PD-: track 7.59 -> 8.14 mm
Other:
- outline, holes or cut-outs redrawn
