File: hardware/Qoobinoo_v2.0/Qoobinoo.kicad_sch (KiCad schematic)
At the start: 32 parts, among them J1 USB_C_Receptacle_USB2.0, J2 Conn_01x02, J3 Conn_01x12, J4 Conn_01x12, SW1 SW_Push, SW2 SW_Push, U1 ATmega32U4-M, X1 16MHz

Commit message: Change USB
Parts:
- removed J1: USB_C_Receptacle_USB2.0, Moldex-21699:Molex-216990_GCT-USB45xx_HRO-TYPE-C-31-M-13x, symbol Connector:USB_C_Receptacle_USB2.0
- removed J2: Conn_01x02, Pin:Pins_USB, symbol Connector_Generic:Conn_01x02
- added J2: Conn_01x02_Female, Pin:Pins_1x02, symbol Connector:Conn_01x02_Female
- added P1: USB_C_Plug_USB2.0, Connector_USB:USB_C_Receptacle_CNCTech_C-ARA1-AK51X, symbol Connector:USB_C_Plug_USB2.0
- C3, C4, C5, C6, C7, C8: footprint Capacitor_SMD:C_0805_2012Metric -> Capacitor_SMD:C_1206_3216Metric
- R1, R10, R2, R3, R6, R7, R8, R9: footprint Resistor_SMD:R_0805_2012Metric -> Resistor_SMD:R_1206_3216Metric
Connections:
- net D+: now also J2.1 (Pin_1), P1.A6 (D+)
- net D-: now also J2.2 (Pin_2), P1.A7 (D-)
- net GND: now also P1.A1 (GND), P1.A12 (GND), P1.B1 (GND), P1.B12 (GND)
- net at F1.1: now also P1.A4 (VBUS), P1.A9 (VBUS), P1.B4 (VBUS), P1.B9 (VBUS)
- no-connect marks 7 -> 5
